File: 7.0/projects/projet_led/projet_led.kicad_pcb (KiCad board)
At the start: 2 copper layers, 80 x 50 mm, 17 parts, among them SW1 SW_Push, SW2 SW_Push, SW3 SW_Push, U1 ATmega32-16P

Commit message: adding some extra backup for rl
Parts:
- removed D6, D7, D8: LD271, LED_THT:LED_D5.0mm_IRGrey
- added R6: 30K, Resistor_THT:R_Axial_DIN0309_L9.0mm_D3.2mm_P12.70mm_Horizontal, F.Cu at (59.5, -25.6)
- added R7: 30K, Resistor_THT:R_Axial_DIN0309_L9.0mm_D3.2mm_P12.70mm_Horizontal, F.Cu at (64.6, -12.9)
- moved U1 113.7 mm to (78.6, 50.6), turned to -90 degrees
- moved D5 20.5 mm to (50.6, -40.8)
Connections:
- D5 pad 2: unconnected-(D5-A-Pad2) -> /chepe
- U1 pad 11: Net-(U1-GND-Pad11) -> GND
- U1 pad 31: Net-(U1-GND-Pad11) -> GND
- U1 pad 40: +1V5 -> unconnected-(U1-PA0-Pad40)
