File: 7.0/projects/projet_led/projet_led.kicad_sch (KiCad schematic)
At the start: 13 parts, among them SW1 SW_Push, SW2 SW_Push, SW3 SW_Push, U1 ATmega32-16P

Commit message: adding some extra backup for rl
Parts:
- added C1, C2: 22pF, symbol Device:C
- added C3: 100nF, symbol Device:C
- added D5: LD271, LED_THT:LED_D5.0mm_IRGrey, symbol LED:LD271
- added R6, R7: 30K, Resistor_THT:R_Axial_DIN0309_L9.0mm_D3.2mm_P12.70mm_Horizontal, symbol Device:R
- added Y1: Crystal, symbol Device:Crystal
Connections:
- net +1V5: no longer U1.40 (PA0)
- net GND: now also U1.11 (GND), U1.31 (GND)
- new net MANGO: R6.1, R7.1
- new net chepe: D5.2 (A), R6.2, R7.2
Other:
- moved on the sheet: D1, D2, D3, D4, R1, R2
